File: hackerhotel-2024-hardware.kicad_sch (KiCad schematic)
At the start: 0 parts

Commit message: Add USB-C, Power regulator and the basics for the RP2040
Parts:
- added C? (x9): 100n, symbol Device:C
- added C? (x2): 1u, symbol Device:C
- added C? (x2): 10u, symbol Device:C
- added C?: 10n, symbol Device:C
- added C? (x2): 10p, symbol Device:C
- added C? (x2): 10uF, symbol Device:C
- added D?: RED, symbol Device:LED
- added D?: 3A/10V/280mV, symbol Device:D_Schottky
- added F?: 6V 0.5A, symbol Device:Fuse
- added FB?: 120R@100Mhz, Resistor_SMD:R_0402_1005Metric, symbol Device:FerriteBead
- added J?: USB_C_Receptacle_USB2.0, symbol Connector:USB_C_Receptacle_USB2.0
- added R? (x2): 1K, symbol Device:R
- added R? (x2): 5K1, symbol Device:R
- added SW?: Bootsel, symbol Switch:SW_Push
- added U?: RP2040, Package_DFN_QFN:QFN-56-1EP_7x7mm_P0.4mm_EP3.2x3.2mm, symbol MCU_RaspberryPi:RP2040
- added U?: W25Q128JVS, Package_SO:SOIC-8_5.23x5.23mm_P1.27mm, symbol Memory_Flash:W25Q128JVS
- added U?: AP2112K-3.3, Package_TO_SOT_SMD:SOT-23-5, symbol Regulator_Linear:AP2112K-3.3
- added Y?: 16Mhz, symbol Device:Crystal_GND24
Connections:
- new net: C?.1, C?.1, FB?.1, U?.43 (ADC_AVDD)
- new net: C?.1, U?.21 (XOUT), Y?.3
- new net: R?.1, SW?.2
- new net: C?.1, D?.1 (K), U?.1 (VIN), U?.3 (EN)
- new net: D?.2 (A), F?.2
- new net: J?.A5 (CC1), R?.1
- new net: J?.B5 (CC2), R?.1
- new net +1V1: C?.1, C?.1, U?.23 (DVDD), U?.45 (VREG_VOUT), U?.50 (DVDD)
- new net +3V3: C?.1, C?.1, C?.1, C?.1, C?.1, C?.1, C?.1, C?.1, C?.1, C?.1, C?.1, FB?.2, R?.1, U?.1 (IOVDD), U?.10 (IOVDD), U?.22 (IOVDD), U?.33 (IOVDD), U?.42 (IOVDD), U?.44 (VREG_IN), U?.48 (USB_VDD), U?.49 (IOVDD), U?.5 (VOUT), U?.8 (VCC)
- new net GND: C?.1, C?.2, C?.2, C?.2, C?.2, C?.2, C?.2, C?.2, C?.2, C?.2, C?.2, C?.2, C?.2, C?.2, C?.2, C?.2, C?.2, C?.2, C?.2, D?.1 (K), J?.A1 (GND), J?.A12 (GND), J?.B1 (GND), J?.B12 (GND), R?.2, R?.2, SW?.1, U?.19 (TESTEN), U?.20 (XIN), U?.4 (GND), U?.57 (GND), Y?.1, Y?.2, Y?.4
- new net PWR_LED_K: D?.2 (A), R?.2
- new net QSPI_SCLK: U?.52 (QSPI_SCLK), U?.6 (CLK)
- new net QSPI_SD0: U?.5 (DI(IO0)), U?.53 (QSPI_SD0)
- new net QSPI_SD1: U?.2 (DO(IO1)), U?.55 (QSPI_SD1)
- new net QSPI_SD2: U?.3 (IO2), U?.54 (QSPI_SD2)
- new net QSPI_SD3: U?.51 (QSPI_SD3), U?.7 (IO3)
- new net QSPI_SS: R?.2, U?.1 (~{CS}), U?.56 (QSPI_SS)
- new net USB_D+: J?.A6 (D+), J?.B6 (D+)
- new net USB_D-: J?.A7 (D-), J?.B7 (D-)
- new net VBUS: F?.1, J?.A4 (VBUS), J?.A9 (VBUS), J?.B4 (VBUS), J?.B9 (VBUS)
- no-connect marks 0 -> 3
Other:
- note added: "ADC_AVDD Filtering"
- note added: "CL = (Cload - Cstray) * 2; CL = 10pF, Cs =~ 5pF"
- note added: "Decoupling DVDD 100n per pin"
- note added: "Decoupling IOVDD, USB_VDD, VREG_IN 100n per pin, 10u chip"
- note added: "Hacker Hotel 2024 Badge"
- note added: "Power Regulator"
- note added: "RP2040"
- note added: "RP2040 Flash Memory (16Mb)"
- note added: "USB-C Receptacle"
- note added: "VBUS from USB, 5V nom. Regulator with power indicator led Can supply 600ma at 3.3v"
- company: (none) -> badge.team
- title: (none) -> Hacker Hotel Badge 2024

Commit message: Add usb hub and wireup the usb ports
Parts:
- added C? (x11): 100n, symbol Device:C
- added C? (x4): 10u, symbol Device:C
- added C? (x2): 1p, symbol Device:C
- added R? (x2): 50K, symbol Device:R
- added R? (x3): 100K, symbol Device:R
- added R? (x2): 10K, symbol Device:R
- added R?: 5K6, symbol Device:R
- added R?: 12K, symbol Device:R
- added SW?: Reset, symbol Switch:SW_Push
- added SW?: SPI boot, symbol Switch:SW_Push
- added U?: USB2412-DZK, QFN28_5X5MC_MCH, symbol Microchip USB2412:USB2412-DZK
- added U?: ESP32-C6-WROOM-1, Espressif:ESP32-C6-WROOM-1, symbol PCM_Espressif:ESP32-C6-WROOM-1
- added Y?: Crystal_GND24, symbol Device:Crystal_GND24
- Y?: LCSC_Part (none) -> C112972
Connections:
- net +1V1: now also C?.1
- net +3V3: now also C?.1, C?.1, C?.1, C?.1, C?.1, C?.1, C?.1, C?.1, C?.1, R?.1, R?.1, R?.1, R?.1, R?.2, U?.10 (VDD33), U?.14 (VDD33), U?.2 (3V3), U?.20 (VDD33), U?.27 (VDD33), U?.4 (VDD33)
- net GND: now also U?.2 (GND), C?.2, C?.2, C?.2, C?.2, C?.2, C?.2, C?.2, C?.2, C?.2, C?.2, C?.2, C?.2, C?.2, C?.2, C?.2, C?.2, R?.1, R?.2, R?.2, SW?.1, SW?.2, U?.1 (GND), U?.12 (GPIO11), U?.15 (TEST1), U?.28 (GND), U?.29 (EPAD), U?.29 (GND), Y?.2, Y?.4
- net USB_D+: now also U?.22 (USBDP_UP)
- net USB_D-: now also U?.21 (USBDM_UP)
- net VBUS: now also C?.1, R?.2, R?.2
- net at C?.1, C?.1, FB?.1: no longer U?.43 (ADC_AVDD)
- net USB_P1_D-: now reaches U?.46 (USB_DM)
- net USB_P1_D-: now also U?.28 (USBDM_DN1)
- net USB_P1_D+: now reaches U?.47 (USB_DP)
- net USB_P1_D+: now also U?.1 (USBDP_DN1)
- new net: R?.2, U?.19 (SUSP_IND/NON_REM0)
- new net: C?.1, R?.2, SW?.2, U?.3 (EN/CHIP_PU)
- new net: R?.2, U?.13 (NON_REMI)
- new net: R?.1, U?.16 (HS_IND)
- new net: R?.1, U?.18 (VBUS_DET)
- new net: R?.1, U?.26 (RBIAS)
- new net: R?.2, U?.10 (GPIO8)
- new net: SW?.1, U?.15 (GPIO9)
- new net: C?.1, Y?.3
- new net CRFILT: C?.1, U?.9 (CRFILT)
- new net PLLFILT: C?.1, U?.25 (PLLFILT)
- new net RESET_N: C?.1, R?.1, U?.17 (RESET_N)
- new net USB2412_XIN: C?.1, U?.24 (XTALIN/CLKIN), Y?.1
- new net USB2412_XOUT: U?.23 (XTALOUT)
- new net USB_P2_D+: U?.14 (GPIO13/USB_D+), U?.3 (USBDP_DN2)
- new net USB_P2_D-: U?.13 (GPIO12/USB_D-), U?.2 (USBDM_DN2)
- no-connect marks 3 -> 8
Other:
- note added: "Decoupling VDD33 100n per pin, 10u chip"
- note added: "Decoupling VREG_VOUT, VREG_VIN 1p per pin"
- note added: "Delay EN with RC See datasheet"
- note added: "ESP32-C6"
- note added: "GPIO8 and GPIO9 control bootmode"
- note added: "Power consumption: 16.6 mA + 35.6 mA + 2.0 mA + 25 mA=~ 80 mA (See popcorn and bootsel in datasheet RP2040, chip_erase in flash datasheet)"
- note added: "Power consumption: 382 mA peak / 120mA 802.15.4 (peak TX WiFi / 802.15.4 @ 0 dBm see datasheet)"
- note added: "TODO: Check resistors for USB on RP2040 in datasheet The USB hub needs a better symbol"
- note added: "USB 2-port hub"
- moved on the sheet: C?, FB?, R?, SW?, U?, Y?

Commit message: Add a part reference
Parts:
- U?: LCSC Part (none) -> C220647
Changed lines of the file:
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@@
       (effects (font (size 1.27 1.27) italic) hide)
     )
-    (property "Field4" "" (at 255.27 151.13 0)
+    (property "LCSC Part" "C220647" (at 255.27 151.13 0)
       (effects (font (size 1.27 1.27)) hide)
     )
