File: hackerhotel-2024-hardware.kicad_pcb (KiCad board)
At the start: 0 parts

Commit message: V1 of schematic
Parts:
- added REF**: TM-2022-2, BamboulabFootprints:TM-2022-2, B.Cu at (133.0, 146.9)
- added REF**: TM-2022-2, BamboulabFootprints:TM-2022-2, B.Cu at (146.0, 146.9)
- added REF**: TM-2022-2, BamboulabFootprints:TM-2022-2, B.Cu at (107.0, 146.9)
- added REF**: TM-2022-2, BamboulabFootprints:TM-2022-2, B.Cu at (94.0, 146.9)
- added REF**: TM-2022-2, BamboulabFootprints:TM-2022-2, B.Cu at (120.0, 146.9)
Other:
- copper layers 0 -> 2
