File: hackerhotel-2024-hardware-renze/_autosave-powermanagement.kicad_sch (KiCad schematic)
At the start: 28 parts, among them J1 Battery, Q2 AP2302B, SW6 SW_SPDT, U1 SY8079AAC, U2 XT4054K421MR-G, U3 SY6280AAC

Commit message: routing almost finished
Parts:
- SW6: footprint (none) -> Button_Switch_SMD:SW_SPDT_PCM12
Changed lines of the file:
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@@
       (effects (font (size 1.27 1.27)))
     )
-    (property "Footprint" "" (at 180.34 49.53 0)
+    (property "Footprint" "Button_Switch_SMD:SW_SPDT_PCM12" (at 180.34 49.53 0)
       (effects (font (size 1.27 1.27)) hide)
     )
