File: hackerhotel-2024-hardware-renze/epaper.kicad_sch (KiCad schematic)
At the start: 18 parts, among them J6 E-Paper, Q2 AP2302B

Commit message: Routing and BOM completed, missing art and regulator update
Parts:
- C1: LCSC C107372 -> C376929; Link (none) -> https://www.lcsc.com/product-detail/Multilayer-Ceramic-Capa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
- C1: LCSC C368809 -> C2918489; Link (none) -> https://www.lcsc.com/product-detail/Multilayer-Ceramic-Capa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
- D2, D3, D4: value NSVR0320MW2T1G -> NSR0320MW2T1G; LCSC C232573 -> C48192; Link (none) -> https://www.lcsc.com/product-detail/Schottky-Barrier-Diodes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
- J6: Link (none) -> https://www.lcsc.com/product-detail/FFC-FPC-Connectors_HRS-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
- L2: Link (none) -> https://www.lcsc.com/product-detail/Power-Inductors_TDK-NLC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
- Q2: Link (none) -> https://www.lcsc.com/product-detail/MOSFETs_ALLPOWER-ShenZh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
- R12: LCSC C25156 -> C2907314; Link (none) -> https://www.lcsc.com/product-detail/Chip-span-style-backgro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
- R12: LCSC C102746 -> C2907288; Link (none) -> https://www.lcsc.com/product-detail/Chip-span-style-backgro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
