File: hackerhotel-2024-hardware-renze/powermanagement.kicad_sch (KiCad schematic)
At the start: 28 parts, among them J1 Battery, Q2 AP2302B, SW6 SW_SPDT, U1 SY8079AAC, U2 XT4054K421MR-G, U3 SY6280AAC

Commit message: Added artwork + more routing
Parts:
- SW6: footprint (none) -> Button_Switch_SMD:SW_SPDT_PCM12
Changed lines of the file:
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@@
+      (effects (font (size 1.27 1.27)) hide)
+    )
+    (property "Field-1" "" (at 200.025 135.89 0)
       (effects (font (size 1.27 1.27)) hide)
     )
@@
     )
     (property "Sponsored" "" (at 104.14 135.89 0)
+      (effects (font (size 1.27 1.27)) hide)
+    )
+    (property "Field-1" "" (at 104.14 135.89 0)
       (effects (font (size 1.27 1.27)) hide)
     )
@@
       (effects (font (size 1.27 1.27)) hide)
     )
+    (property "Field-1" "" (at 177.8 69.85 0)
+      (effects (font (size 1.27 1.27)) hide)
+    )
     (pin "1")
     (pin "2")
@@
       (effects (font (size 1.27 1.27)) hide)
     )
+    (property "Field-1" "" (at 109.855 76.2 0)
+      (effects (font (size 1.27 1.27)) hide)
+    )
     (pin "1")
     (pin "2")
@@
     )
     (property "Sponsored" "" (at 208.28 58.42 0)
+      (effects (font (size 1.27 1.27)) hide)
+    )
+    (property "Field-1" "" (at 208.28 58.42 0)
       (effects (font (size 1.27 1.27)) hide)
     )
@@
       (effects (font (size 1.27 1.27)) hide)
     )
+    (property "Field-1" "" (at 97.155 71.12 0)
+      (effects (font (size 1.27 1.27)) hide)
+    )
     (pin "1")
     (pin "2")
@@
       (effects (font (size 1.27 1.27)))
     )
-    (property "Footprint" "" (at 180.34 49.53 0)
+    (property "Footprint" "Button_Switch_SMD:SW_SPDT_PCM12" (at 180.34 49.53 0)
       (effects (font (size 1.27 1.27)) hide)
     )
@@
       (effects (font (size 1.27 1.27)) hide)
     )
+    (property "Field-1" "" (at 180.34 49.53 0)
+      (effects (font (size 1.27 1.27)) hide)
+    )
     (pin "3")
     (pin "1")
@@
       (effects (font (size 1.27 1.27)) hide)
     )
+    (property "Field-1" "" (at 171.45 66.04 0)
+      (effects (font (size 1.27 1.27)) hide)
+    )
     (pin "1")
     (pin "2")
@@
       (effects (font (size 1.27 1.27)) hide)
     )
+    (property "Field-1" "" (at 219.71 66.04 0)
+      (effects (font (size 1.27 1.27)) hide)
+    )
     (pin "1")
     (pin "2")
@@
     )
     (property "Sponsored" "" (at 189.865 125.73 0)
+      (effects (font (size 1.27 1.27)) hide)
+    )
+    (property "Field-1" "" (at 189.865 125.73 0)
       (effects (font (size 1.27 1.27)) hide)
     )
@@
     )
     (property "Sponsored" "" (at 84.455 66.04 0)
+      (effects (font (size 1.27 1.27)) hide)
+    )
+    (property "Field-1" "" (at 84.455 66.04 0)
       (effects (font (size 1.27 1.27)) hide)
     )
@@
       (effects (font (size 1.27 1.27)) hide)
     )
+    (property "Field-1" "" (at 187.96 58.42 0)
+      (effects (font (size 1.27 1.27)) hide)
+    )
     (pin "1")
     (pin "2")
@@
       (effects (font (size 1.27 1.27)) hide)
     )
+    (property "Field-1" "" (at 62.865 76.2 0)
+      (effects (font (size 1.27 1.27)) hide)
+    )
     (pin "1")
     (pin "2")
@@
     )
     (property "Sponsored" "" (at 189.23 50.8 0)
+      (effects (font (size 1.27 1.27)) hide)
+    )
+    (property "Field-1" "" (at 189.23 50.8 0)
       (effects (font (size 1.27 1.27)) hide)
     )
@@
       (effects (font (size 1.27 1.27)) hide)
     )
+    (property "Field-1" "" (at 170.18 134.62 0)
+      (effects (font (size 1.27 1.27)) hide)
+    )
     (pin "1")
     (pin "2")
@@
       (effects (font (size 1.27 1.27)) hide)
     )
+    (property "Field-1" "" (at 116.84 130.81 0)
+      (effects (font (size 1.27 1.27)) hide)
+    )
     (pin "1")
     (pin "2")
@@
     )
     (property "Sponsored" "" (at 71.755 76.2 0)
+      (effects (font (size 1.27 1.27)) hide)
+    )
+    (property "Field-1" "" (at 71.755 76.2 0)
       (effects (font (size 1.27 1.27)) hide)
     )
@@
       (effects (font (size 1.27 1.27)) hide)
     )
+    (property "Field-1" "" (at 97.155 66.04 0)
+      (effects (font (size 1.27 1.27)) hide)
+    )
     (pin "1")
     (pin "2")
@@
       (effects (font (size 1.27 1.27)) hide)
     )
+    (property "Field-1" "" (at 154.94 135.89 0)
+      (effects (font (size 1.27 1.27)) hide)
+    )
     (pin "1")
     (pin "2")
@@
       (effects (font (size 1.27 1.27)) hide)
     )
+    (property "Field-1" "" (at 97.155 63.5 0)
+      (effects (font (size 1.27 1.27)) hide)
+    )
     (pin "1")
     (pin "2")
@@
       (effects (font (size 1.27 1.27)) hide)
     )
+    (property "Field-1" "" (at 93.98 135.89 0)
+      (effects (font (size 1.27 1.27)) hide)
+    )
     (pin "1")
     (pin "2")
@@
       (effects (font (size 1.27 1.27)) hide)
     )
+    (property "Field-1" "" (at 208.28 44.45 0)
+      (effects (font (size 1.27 1.27)) hide)
+    )
     (pin "1")
     (pin "2")
@@
       (effects (font (size 1.27 1.27)) hide)
     )
+    (property "Field-1" "" (at 171.45 74.93 0)
+      (effects (font (size 1.27 1.27)) hide)
+    )
     (pin "1")
     (pin "2")
@@
       (effects (font (size 1.27 1.27)) hide)
     )
+    (property "Field-1" "" (at 117.475 76.2 0)
+      (effects (font (size 1.27 1.27)) hide)
+    )
     (pin "1")
     (pin "2")
@@
       (effects (font (size 1.27 1.27)) hide)
     )
+    (property "Field-1" "" (at 92.075 76.2 0)
+      (effects (font (size 1.27 1.27)) hide)
+    )
     (pin "1")
     (pin "2")
@@
       (effects (font (size 1.27 1.27)) hide)
     )
+    (property "Field-1" "" (at 148.59 123.19 0)
+      (effects (font (size 1.27 1.27)) hide)
+    )
     (pin "1")
     (pin "2")
@@
     )
     (property "Sponsored" "" (at 189.865 135.89 0)
+      (effects (font (size 1.27 1.27)) hide)
+    )
+    (property "Field-1" "" (at 189.865 135.89 0)
       (effects (font (size 1.27 1.27)) hide)
     )
@@
       (effects (font (size 1.27 1.27)) hide)
     )
+    (property "Field-1" "" (at 130.81 128.27 0)
+      (effects (font (size 1.27 1.27)) hide)
+    )

Commit message: Routing and BOM completed, missing art and regulator update
Parts:
- C1, C7: LCSC C15525 -> C5189822; Link (none) -> https://www.lcsc.com/product-detail/Multilayer-Ceramic-Capa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
- C13, C2, C3: LCSC C307331 -> C476766; Link (none) -> https://www.lcsc.com/product-detail/Multilayer-Ceramic-Capa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
- C4, C6, C8: Link (none) -> https://www.lcsc.com/product-detail/Multilayer-Ceramic-Capa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
- C5: LCSC C466226 -> C5137614; Link (none) -> https://www.lcsc.com/product-detail/Multilayer-Ceramic-Capa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
- D1: value NSVR0320MW2T1G -> NSR0320MW2T1G; LCSC C232573 -> C48192; Link (none) -> https://www.lcsc.com/product-detail/Schottky-Barrier-Diodes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
- J1: Link (none) -> https://www.lcsc.com/product-detail/Wire-To-Board-Wire-To-W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
- L1: Link (none) -> https://www.lcsc.com/product-detail/Power-Inductors_PSA-Pro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
- Q2: Link (none) -> https://www.lcsc.com/product-detail/MOSFETs_ALLPOWER-ShenZh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
- R11: LCSC C3017479 -> C3017842; Link (none) -> https://www.lcsc.com/product-detail/Chip-span-style-backgro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
- R12, R13: LCSC C25741 -> C2907293; Link (none) -> https://www.lcsc.com/product-detail/Chip-span-style-backgro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
- R14: LCSC C25900 -> C2907326; Link (none) -> https://www.lcsc.com/product-detail/Chip-span-style-backgro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
- R3: LCSC C25552 -> C3017846; Link (none) -> https://www.lcsc.com/product-detail/Chip-span-style-backgro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
- R5, R7, R8: LCSC C25744 -> C5140188; Link (none) -> https://www.lcsc.com/product-detail/Chip-span-style-backgro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
- R6: LCSC C26980 -> C5266157; Link (none) -> https://www.lcsc.com/product-detail/Chip-span-style-backgro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
- R8: LCSC C25744 -> C2907293; Link (none) -> https://www.lcsc.com/product-detail/Chip-span-style-backgro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
- SW6: LCSC (none) -> C319020; Link (none) -> https://www.lcsc.com/product-detail/Toggle-Switches_XKB-Con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
- U1: Link (none) -> https://www.lcsc.com/product-detail/DC-DC-Converters_Silerg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
- U2: Link (none) -> https://www.lcsc.com/product-detail/Battery-Management-ICs_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
- U3: Link (none) -> https://www.lcsc.com/product-detail/Power-Distribution-Swit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
