File: hackerhotel-2024-hardware-renze/hh2024.kicad_sch (KiCad schematic)
At the start: 55 parts, among them J1 SAO, J2 Breakout pads, J3 Micro_SD_Card, J4 USB-C, K1 SANYOU_SRD_Form_C, Q3 AP2302B, SW1 Multi-Directional-Switches, SW2 Multi-Directional-Switches, SW3 Multi-Directional-Switches, SW4 Multi-Directional-Switches, SW5 Multi-Directional-Switches, U5 CH32V003F4U6

Commit message: before tidy
Other:
- note added: "A"
- note added: "B"
- note added: "D"
- note added: "E"
- note added: "F"
- note added: "G"
- note added: "H"
- note added: "I"
- note added: "K"
- note added: "L"
- note added: "M"
- note added: "N"
- note added: "O"
- note added: "P"
- note added: "R"
- note added: "S"
- note added: "T"
- note added: "V"
- note added: "W"
- note added: "Y"
Changed lines of the file:
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@@
     (stroke (width 0) (type default))
+  )
+  (text "F" (exclude_from_sim no)
+ (at 51.308 98.298 0)
+    (effects (font (size 1.27 1.27)))
+  )
+  (text "V" (exclude_from_sim no)
+ (at 81.788 105.918 0)
+    (effects (font (size 1.27 1.27)))
+  )
+  (text "P" (exclude_from_sim no)
+ (at 91.948 90.678 0)
+    (effects (font (size 1.27 1.27)))
+  )
+  (text "D" (exclude_from_sim no)
+ (at 82.042 75.438 0)
+    (effects (font (size 1.27 1.27)))
+  )
+  (text "A" (exclude_from_sim no)
+ (at 71.628 75.438 0)
+    (effects (font (size 1.27 1.27)))
+  )
+  (text "M" (exclude_from_sim no)
+ (at 71.628 105.918 0)
+    (effects (font (size 1.27 1.27)))
+  )
+  (text "R" (exclude_from_sim no)
+ (at 91.948 105.918 0)
+    (effects (font (size 1.27 1.27)))
   )
   (text "Top (orange)" (exclude_from_sim no)
  (at 32.512 69.342 0)
+    (effects (font (size 1.27 1.27)))
+  )
+  (text "G" (exclude_from_sim no)
+ (at 61.468 90.678 0)
+    (effects (font (size 1.27 1.27)))
+  )
+  (text "N" (exclude_from_sim no)
+ (at 61.468 105.918 0)
+    (effects (font (size 1.27 1.27)))
+  )
+  (text "Y" (exclude_from_sim no)
+ (at 91.948 83.058 0)
+    (effects (font (size 1.27 1.27)))
+  )
+  (text "S" (exclude_from_sim no)
+ (at 71.628 98.298 0)
+    (effects (font (size 1.27 1.27)))
+  )
+  (text "E" (exclude_from_sim no)
+ (at 71.628 83.058 0)
+    (effects (font (size 1.27 1.27)))
+  )
+  (text "W" (exclude_from_sim no)
+ (at 81.788 98.298 0)
+    (effects (font (size 1.27 1.27)))
+  )
+  (text "T" (exclude_from_sim no)
+ (at 81.788 90.678 0)
+    (effects (font (size 1.27 1.27)))
+  )
+  (text "I" (exclude_from_sim no)
+ (at 51.308 75.438 0)
+    (effects (font (size 1.27 1.27)))
+  )
+  (text "L" (exclude_from_sim no)
+ (at 51.308 83.058 0)
+    (effects (font (size 1.27 1.27)))
+  )
+  (text "H" (exclude_from_sim no)
+ (at 61.468 75.438 0)
     (effects (font (size 1.27 1.27)))
   )
@@
     (effects (font (size 1.27 1.27)))
   )
+  (text "B" (exclude_from_sim no)
+ (at 51.308 90.678 0)
+    (effects (font (size 1.27 1.27)))
+  )
+  (text "O" (exclude_from_sim no)
+ (at 91.948 98.298 0)
+    (effects (font (size 1.27 1.27)))
+  )
+  (text "K\n" (exclude_from_sim no)
+ (at 61.468 83.058 0)
+    (effects (font (size 1.27 1.27)))
+  )
