File: hackerhotel-2024-hardware-renze/microcontroller.kicad_sch (KiCad schematic)
At the start: 8 parts, among them U4 ESP32-C6-WROOM-1

Commit message: Routing and BOM completed, missing art and regulator update
Parts:
- C13: LCSC C307331 -> C476766; Link (none) -> https://www.lcsc.com/product-detail/Multilayer-Ceramic-Capa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
- C9: LCSC C107372 -> C376929; Link (none) -> https://www.lcsc.com/product-detail/Multilayer-Ceramic-Capa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
- R10: LCSC C25744 -> C5140188; Link (none) -> https://www.lcsc.com/product-detail/Chip-span-style-backgro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
- R15, R16: LCSC C25156 -> C2907314; Link (none) -> https://www.lcsc.com/product-detail/Chip-span-style-backgro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
Changed lines of the file:
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@@
       (effects (font (size 1.27 1.27)) hide)
     )
-    (property "Datasheet" "https://datasheet.lcsc.com/lcsc/2110260030_UNI-ROYAL-Uniroyal-Elec-0402WGF1002TCE_C25744.pdf" (at 177.8 57.15 0)
+    (property "Datasheet" "https://datasheet.lcsc.com/lcsc/2208231730_VO-SCR0805J10K_C5140188.pdf" (at 177.8 57.15 0)
       (effects (font (size 1.27 1.27)) hide)
     )
@@
       (effects (font (size 1.27 1.27)) hide)
     )
-    (property "LCSC" "C25744" (at 177.8 57.15 0)
+    (property "LCSC" "C5140188 " (at 177.8 57.15 0)
       (effects (font (size 1.27 1.27)) hide)
     )
@@
       (effects (font (size 1.27 1.27)) hide)
     )
+    (property "Link" "https://www.lcsc.com/product-detail/Chip-span-style-background-color-ff0-Resistor-span-Surface-Mount_VO-SCR0805J10K_C5140188.html" (at 177.8 57.15 0)
+      (effects (font (size 1.27 1.27)) hide)
+    )
     (pin "1")
     (pin "2")
@@
       (effects (font (size 1.27 1.27)) hide)
     )
-    (property "Datasheet" "https://datasheet.lcsc.com/lcsc/2110260030_UNI-ROYAL-Uniroyal-Elec-0402WGF1002TCE_C25744.pdf" (at 90.17 58.42 0)
+    (property "Datasheet" "https://datasheet.lcsc.com/lcsc/2208231730_VO-SCR0805J10K_C5140188.pdf" (at 90.17 58.42 0)
       (effects (font (size 1.27 1.27)) hide)
     )
@@
       (effects (font (size 1.27 1.27)) hide)
     )
-    (property "LCSC" "C25744" (at 90.17 58.42 0)
+    (property "LCSC" "C5140188 " (at 90.17 58.42 0)
       (effects (font (size 1.27 1.27)) hide)
     )
@@
     )
     (property "Field-1" "" (at 90.17 58.42 0)
+      (effects (font (size 1.27 1.27)) hide)
+    )
+    (property "Link" "https://www.lcsc.com/product-detail/Chip-span-style-background-color-ff0-Resistor-span-Surface-Mount_VO-SCR0805J10K_C5140188.html" (at 90.17 58.42 0)
       (effects (font (size 1.27 1.27)) hide)
     )
@@
       (effects (font (size 1.27 1.27)) hide)
     )
-    (property "Datasheet" "https://datasheet.lcsc.com/lcsc/2304140030_Samsung-Electro-Mechanics-CL05B104KB54PNC_C307331.pdf" (at 76.2 58.42 0)
+    (property "Datasheet" "https://datasheet.lcsc.com/lcsc/1912300933_TORCH-C0805B104K500NT_C476766.pdf" (at 76.2 58.42 0)
       (effects (font (size 1.27 1.27)) hide)
     )
@@
       (effects (font (size 1.27 1.27)) hide)
     )
-    (property "LCSC" "C307331" (at 76.2 58.42 0)
+    (property "LCSC" "C476766" (at 76.2 58.42 0)
       (effects (font (size 1.27 1.27)) hide)
     )
@@
     )
     (property "Field-1" "" (at 76.2 58.42 0)
+      (effects (font (size 1.27 1.27)) hide)
+    )
+    (property "Link" "https://www.lcsc.com/product-detail/Multilayer-Ceramic-Capacitors-MLCC-SMD-SMT_TORCH-C0805B104K500NT_C476766.html" (at 76.2 58.42 0)
       (effects (font (size 1.27 1.27)) hide)
     )
@@
       (effects (font (size 1.27 1.27)) hide)
     )
-    (property "Datasheet" "https://datasheet.lcsc.com/lcsc/2304140030_Samsung-Electro-Mechanics-CL05A105KQ5NNNC_C107372.pdf" (at 90.17 78.74 0)
+    (property "Datasheet" "https://datasheet.lcsc.com/lcsc/2304140030_CCTC-TCC0805X7R105M500FT_C376929.pdf" (at 90.17 78.74 0)
       (effects (font (size 1.27 1.27)) hide)
     )
@@
       (effects (font (size 1.27 1.27)) hide)
     )
-    (property "LCSC" "C107372" (at 90.17 78.74 0)
+    (property "LCSC" "C376929" (at 90.17 78.74 0)
       (effects (font (size 1.27 1.27)) hide)
     )
@@
       (effects (font (size 1.27 1.27)) hide)
     )
+    (property "Link" "https://www.lcsc.com/product-detail/Multilayer-Ceramic-Capacitors-MLCC-SMD-SMT_CCTC-TCC0805X7R105M500FT_C376929.html" (at 90.17 78.74 0)
+      (effects (font (size 1.27 1.27)) hide)
+    )
     (pin "1")
     (pin "2")
@@
       (effects (font (size 1.27 1.27)) hide)
     )
-    (property "Datasheet" "https://datasheet.lcsc.com/lcsc/2110260030_UNI-ROYAL-Uniroyal-Elec-0402WGF1002TCE_C25744.pdf" (at 175.26 57.15 0)
+    (property "Datasheet" "https://datasheet.lcsc.com/lcsc/2208231730_VO-SCR0805J10K_C5140188.pdf" (at 175.26 57.15 0)
       (effects (font (size 1.27 1.27)) hide)
     )
@@
       (effects (font (size 1.27 1.27)) hide)
     )
-    (property "LCSC" "C25744" (at 175.26 57.15 0)
+    (property "LCSC" "C5140188 " (at 175.26 57.15 0)
       (effects (font (size 1.27 1.27)) hide)
     )
@@
       (effects (font (size 1.27 1.27)) hide)
     )
+    (property "Link" "https://www.lcsc.com/product-detail/Chip-span-style-background-color-ff0-Resistor-span-Surface-Mount_VO-SCR0805J10K_C5140188.html" (at 175.26 57.15 0)
+      (effects (font (size 1.27 1.27)) hide)
+    )
     (pin "1")
     (pin "2")
@@
       (effects (font (size 1.27 1.27)) hide)
     )
-    (property "Datasheet" "https://datasheet.lcsc.com/lcsc/2205311845_UNI-ROYAL-Uniroyal-Elec-0402WGJ0270TCE_C25156.pdf" (at 185.42 73.66 0)
+    (property "Datasheet" "https://datasheet.lcsc.com/lcsc/2308241947_FOJAN-FRC0805J270-TS_C2907314.pdf" (at 185.42 73.66 0)
       (effects (font (size 1.27 1.27)) hide)
     )
@@
       (effects (font (size 1.27 1.27)) hide)
     )
-    (property "LCSC" "C25156" (at 185.42 73.66 0)
+    (property "LCSC" "C2907314" (at 185.42 73.66 0)
       (effects (font (size 1.27 1.27)) hide)
     )
@@
       (effects (font (size 1.27 1.27)) hide)
     )
+    (property "Link" "https://www.lcsc.com/product-detail/Chip-span-style-background-color-ff0-Resistor-span-Surface-Mount_FOJAN-FRC0805J270-TS_C2907314.html" (at 185.42 73.66 0)
+      (effects (font (size 1.27 1.27)) hide)
+    )
     (pin "1")
     (pin "2")
@@
       (effects (font (size 1.27 1.27)) hide)
     )
-    (property "Datasheet" "https://datasheet.lcsc.com/lcsc/2205311845_UNI-ROYAL-Uniroyal-Elec-0402WGJ0270TCE_C25156.pdf" (at 185.42 71.12 0)
+    (property "Datasheet" "https://datasheet.lcsc.com/lcsc/2308241947_FOJAN-FRC0805J270-TS_C2907314.pdf" (at 185.42 71.12 0)
       (effects (font (size 1.27 1.27)) hide)
     )
@@
       (effects (font (size 1.27 1.27)) hide)
     )
-    (property "LCSC" "C25156" (at 185.42 71.12 0)
+    (property "LCSC" "C2907314" (at 185.42 71.12 0)
       (effects (font (size 1.27 1.27)) hide)
     )
@@
     )
     (property "Field-1" "" (at 185.42 71.12 0)
+      (effects (font (size 1.27 1.27)) hide)
+    )
+    (property "Link" "https://www.lcsc.com/product-detail/Chip-span-style-background-color-ff0-Resistor-span-Surface-Mount_FOJAN-FRC0805J270-TS_C2907314.html" (at 185.42 71.12 0)
       (effects (font (size 1.27 1.27)) hide)
     )
@@
       (effects (font (size 1.27 1.27)) hide)
     )
+    (property "Link" "" (at 144.78 91.44 0)
+      (effects (font (size 1.27 1.27)) hide)
+    )

Commit message: V1 complete
Parts:
- added R13: 100k, Resistor_SMD:R_0805_2012Metric, symbol symbols:R
- added TP2 (x3): TestPoint, TestPoint:TestPoint_Pad_1.0x1.0mm, symbol Connector:TestPoint
Connections:
- net GND: now also R13.1
- net Relay Ctrl: now also U4.23 (GPIO15), R13.2; no longer R10.2, U4.15 (GPIO9)
- net at U4.20 (GPIO22): now also TP2.1
- net at U4.21 (GPIO23): now also TP2.1
- new net: R10.2, TP2.1, U4.15 (GPIO9)
Changed lines of the file:
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@@
     (comment 1 "License: CERN Open Hardware Licence Version 2 - Permissive")
   )
+  (junction (at 201.93 91.44) (diameter 0) (color 0 0 0 0)
+  )
   (junction (at 177.8 86.36) (diameter 0) (color 0 0 0 0)
   )
@@
     (stroke (width 0) (type default))
   )
+  (wire (pts (xy 201.93 91.44) (xy 205.74 91.44))
+    (stroke (width 0) (type default))
+  )
   (wire (pts (xy 172.72 86.36) (xy 177.8 86.36))
     (stroke (width 0) (type default))
@@
     (stroke (width 0) (type default))
   )
+  (wire (pts (xy 201.93 101.6) (xy 201.93 100.33))
+    (stroke (width 0) (type default))
+  )
+  (wire (pts (xy 201.93 92.71) (xy 201.93 91.44))
+    (stroke (width 0) (type default))
+  )
   (wire (pts (xy 177.8 60.96) (xy 177.8 86.36))
     (stroke (width 0) (type default))
   )
+  (wire (pts (xy 173.99 106.68) (xy 172.72 106.68))
+    (stroke (width 0) (type default))
+  )
   (wire (pts (xy 172.72 71.12) (xy 181.61 71.12))
     (stroke (width 0) (type default))
@@
     (stroke (width 0) (type default))
   )
-  (wire (pts (xy 172.72 91.44) (xy 186.69 91.44))
+  (wire (pts (xy 172.72 91.44) (xy 201.93 91.44))
     (stroke (width 0) (type default))
   )
@@
     (effects (font (size 1.27 1.27)) (justify left))
   )
-  (hierarchical_label "Relay Ctrl" (shape output) (at 186.69 86.36 0) (fields_autoplaced)
+  (hierarchical_label "Relay Ctrl" (shape output) (at 205.74 91.44 0) (fields_autoplaced)
     (effects (font (size 1.27 1.27)) (justify left))
   )
@@
     )
   )
+  (symbol (lib_id "symbols2:GND") (at 201.93 101.6 0) (unit 1)
+    (exclude_from_sim no) (in_bom yes) (on_board yes) (dnp no)
+    (property "Reference" "#PWR010" (at 201.93 107.95 0)
+      (effects (font (size 1.27 1.27)) hide)
+    )
+    (property "Value" "GND" (at 202.057 105.9942 0)
+      (effects (font (size 1.27 1.27)))
+    )
+    (property "Footprint" "" (at 201.93 101.6 0)
+      (effects (font (size 1.27 1.27)) hide)
+    )
+    (property "Datasheet" "" (at 201.93 101.6 0)
+      (effects (font (size 1.27 1.27)) hide)
+    )
+    (property "Description" "Power symbol creates a global label with name \"GND\" , ground" (at 201.93 101.6 0)
+      (effects (font (size 1.27 1.27)) hide)
+    )
+    (pin "1")
+    (instances
+      (project "hh2024"
+        (path "/5f312b85-6822-40a3-b417-2df49696ca2d"
+          (reference "#PWR010") (unit 1)
+        )
+        (path "/5f312b85-6822-40a3-b417-2df49696ca2d/6c7d4443-00e2-4496-9768-e5d745979ee2"
+          (reference "#PWR05") (unit 1)
+        )
+      )
+    )
+  )
   (symbol (lib_id "symbols2:GND") (at 144.78 130.81 0) (unit 1)
     (exclude_from_sim no) (in_bom yes) (on_board yes) (dnp no)
@@
         (path "/5f312b85-6822-40a3-b417-2df49696ca2d/6c7d4443-00e2-4496-9768-e5d745979ee2"
           (reference "#PWR028") (unit 1)
+        )
+      )
+    )
+  )
+  (symbol (lib_id "symbols:R") (at 201.93 96.52 180) (unit 1)
+    (exclude_from_sim no) (in_bom yes) (on_board yes) (dnp no)
+    (property "Reference" "R13" (at 205.74 95.25 0)
+      (effects (font (size 1.27 1.27)))
+    )
+    (property "Value" "100k" (at 205.74 97.79 0)
+      (effects (font (size 1.27 1.27)))
+    )
+    (property "Footprint" "Resistor_SMD:R_0805_2012Metric" (at 203.708 96.52 90)
+      (effects (font (size 1.27 1.27)) hide)
+    )
+    (property "Datasheet" "https://datasheet.lcsc.com/lcsc/2308241947_FOJAN-FRC0805J104-TS_C2907293.pdf" (at 201.93 96.52 0)
+      (effects (font (size 1.27 1.27)) hide)
+    )
+    (property "Description" "" (at 201.93 96.52 0)
+      (effects (font (size 1.27 1.27)) hide)
+    )
+    (property "LCSC" "C2907293" (at 201.93 96.52 0)
+      (effects (font (size 1.27 1.27)) hide)
+    )
+    (property "Buy early" "" (at 201.93 96.52 0)
+      (effects (font (size 1.27 1.27)) hide)
+    )
+    (property "Category" "" (at 201.93 96.52 0)
+      (effects (font (size 1.27 1.27)) hide)
+    )
+    (property "MANUFACTURER" "" (at 201.93 96.52 0)
+      (effects (font (size 1.27 1.27)) hide)
+    )
+    (property "MPN" "" (at 201.93 96.52 0)
+      (effects (font (size 1.27 1.27)) hide)
+    )
+    (property "Manufacturer" "" (at 201.93 96.52 0)
+      (effects (font (size 1.27 1.27)) hide)
+    )
+    (property "Mouser" "" (at 201.93 96.52 0)
+      (effects (font (size 1.27 1.27)) hide)
+    )
+    (property "Price" "" (at 201.93 96.52 0)
+      (effects (font (size 1.27 1.27)) hide)
+    )
+    (property "Quantity" "" (at 201.93 96.52 0)
+      (effects (font (size 1.27 1.27)) hide)
+    )
+    (property "Sponsored" "" (at 201.93 96.52 0)
+      (effects (font (size 1.27 1.27)) hide)
+    )
+    (property "Field-1" "" (at 201.93 96.52 0)
+      (effects (font (size 1.27 1.27)) hide)
+    )
+    (property "Link" "https://www.lcsc.com/product-detail/Chip-span-style-background-color-ff0-Resistor-span-Surface-Mount_FOJAN-FRC0805J104-TS_C2907293.html" (at 201.93 96.52 0)
+      (effects (font (size 1.27 1.27)) hide)
+    )
+    (pin "1")
+    (pin "2")
+    (instances
+      (project "hh2024"
+        (path "/5f312b85-6822-40a3-b417-2df49696ca2d"
+          (reference "R13") (unit 1)
+        )
+        (path "/5f312b85-6822-40a3-b417-2df49696ca2d/77fdc604-e080-44e7-9e66-e31abda69ba3"
+          (reference "R18") (unit 1)
+        )
+        (path "/5f312b85-6822-40a3-b417-2df49696ca2d/6c7d4443-00e2-4496-9768-e5d745979ee2"
+          (reference "R32") (unit 1)
         )
       )
@@
     )
   )
+  (symbol (lib_id "Connector:TestPoint") (at 173.99 104.14 270) (unit 1)
+    (exclude_from_sim no) (in_bom yes) (on_board yes) (dnp no)
+    (property "Reference" "TP2" (at 182.118 104.14 90)
+      (effects (font (size 1.27 1.27)) (justify right))
+    )
+    (property "Value" "TestPoint" (at 181.102 112.776 0)
+      (effects (font (size 1.27 1.27)) (justify right) hide)
+    )
+    (property "Footprint" "TestPoint:TestPoint_Pad_1.0x1.0mm" (at 173.99 109.22 0)
+      (effects (font (size 1.27 1.27)) hide)
+    )
+    (property "Datasheet" "~" (at 173.99 109.22 0)
+      (effects (font (size 1.27 1.27)) hide)
+    )
+    (property "Description" "test point" (at 173.99 104.14 0)
+      (effects (font (size 1.27 1.27)) hide)
+    )
+    (pin "1")
+    (instances
+      (project "hh2024"
+        (path "/5f312b85-6822-40a3-b417-2df49696ca2d"
+          (reference "TP2") (unit 1)
+        )
+        (path "/5f312b85-6822-40a3-b417-2df49696ca2d/6c7d4443-00e2-4496-9768-e5d745979ee2"
+          (reference "TP4") (unit 1)
+        )
+      )
+    )
+  )
   (symbol (lib_id "symbols2:GND") (at 90.17 82.55 0) (unit 1)
     (exclude_from_sim no) (in_bom yes) (on_board yes) (dnp no)
@@
         (path "/5f312b85-6822-40a3-b417-2df49696ca2d/6c7d4443-00e2-4496-9768-e5d745979ee2"
           (reference "#PWR025") (unit 1)
+        )
+      )
+    )
+  )
+  (symbol (lib_id "Connector:TestPoint") (at 186.69 86.36 270) (unit 1)
+    (exclude_from_sim no) (in_bom yes) (on_board yes) (dnp no)
+    (property "Reference" "TP2" (at 194.564 86.614 90)
+      (effects (font (size 1.27 1.27)) (justify right))
+    )
+    (property "Value" "TestPoint" (at 193.802 94.996 0)
+      (effects (font (size 1.27 1.27)) (justify right) hide)
+    )
+    (property "Footprint" "TestPoint:TestPoint_Pad_1.0x1.0mm" (at 186.69 91.44 0)
+      (effects (font (size 1.27 1.27)) hide)
+    )
+    (property "Datasheet" "~" (at 186.69 91.44 0)
+      (effects (font (size 1.27 1.27)) hide)
+    )
+    (property "Description" "test point" (at 186.69 86.36 0)
+      (effects (font (size 1.27 1.27)) hide)
+    )
+    (pin "1")
+    (instances
+      (project "hh2024"
+        (path "/5f312b85-6822-40a3-b417-2df49696ca2d"
+          (reference "TP2") (unit 1)
+        )
+        (path "/5f312b85-6822-40a3-b417-2df49696ca2d/6c7d4443-00e2-4496-9768-e5d745979ee2"
+          (reference "TP3") (unit 1)
         )
       )
@@
         )
       )
+    )
+  )
+  (symbol (lib_id "Connector:TestPoint") (at 173.99 106.68 270) (unit 1)
+    (exclude_from_sim no) (in_bom yes) (on_board yes) (dnp no)
+    (property "Reference" "TP2" (at 182.372 106.934 90)
+      (effects (font (size 1.27 1.27)) (justify right))
+    )
+    (property "Value" "TestPoint" (at 181.102 115.316 0)
+      (effects (font (size 1.27 1.27)) (justify right) hide)
+    )
+    (property "Footprint" "TestPoint:TestPoint_Pad_1.0x1.0mm" (at 173.99 111.76 0)
+      (effects (font (size 1.27 1.27)) hide)
+    )
+    (property "Datasheet" "~" (at 173.99 111.76 0)
+      (effects (font (size 1.27 1.27)) hide)
+    )
+    (property "Description" "test point" (at 173.99 106.68 0)
+      (effects (font (size 1.27 1.27)) hide)
+    )
+    (pin "1")
+    (instances
+      (project "hh2024"
+        (path "/5f312b85-6822-40a3-b417-2df49696ca2d"
+          (reference "TP2") (unit 1)
+        )
+        (path "/5f312b85-6822-40a3-b417-2df49696ca2d/6c7d4443-00e2-4496-9768-e5d745979ee2"
+          (reference "TP5") (unit 1)
+        )
+      )

Commit message: before tidy
Connections:
- net GPIO9: now reaches R10.2, TP2.1, U4.15 (GPIO9)
Changed lines of the file:
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@@
     (effects (font (size 1.27 1.27)) (justify left top))
+  )
+  (label "GPIO9" (at 179.07 86.36 0) (fields_autoplaced)
+    (effects (font (size 1.27 1.27)) (justify left bottom))
   )
   (hierarchical_label "SAO IO2" (shape bidirectional) (at 116.84 71.12 180) (fields_autoplaced)
